Commit message: turned joint to torso to head to fixed

File: config/gazebo_hera.urdf (robot description, URDF)
Before this commit: robot hera, 27 links, 26 joints
Joints:
- joint joint_torso_to_head: type revolute -> fixed

Commit message: added new controller for all motors and new point pose

File: config/gazebo_hera.urdf (robot description, URDF)
Before this commit: robot hera, 27 links, 26 joints
Links:
- removed link xtion
- removed link xtion_depth
- removed link xtion_optical
- added link xtion_link, mass 0.01; collision box size=0.04 0.18 0.07; visual mesh filename=package://hera_description/meshes/asus_xtion.stl
- added link xtion_link_depth
- added link xtion_link_optical
Joints:
- removed joint joint_torso_to_xtion
- removed joint joint_xtion_to_xtion_depth
- removed joint joint_xtion_to_xtion_otptical
- added joint joint_torso_to_xtion_link: type fixed, parent torso, child xtion_link, origin xyz=0.215 0 -0.17 rpy=0 0 0
- added joint joint_xtion_link_to_xtion_link_depth: type fixed, parent xtion_link, child xtion_link_depth, origin xyz=0.0 0.049 0.016 rpy=0 0 0
- added joint joint_xtion_link_to_xtion_link_otptical: type fixed, parent xtion_link, child xtion_link_optical, origin xyz=0 0 0 rpy=-1.5707963267948966 0 -1.5707963267948966
- joint elbow_pan_joint: limit lower=-0.8 upper=0.8 effort=0 velocity=5 -> lower=-1.57 upper=1.57 effort=0 velocity=5
- joint joint_torso_to_torso_sensor_plat: limit lower=-1.0 upper=0.45 effort=30 velocity=0.5 -> lower=-1.5 upper=0.1 effort=30 velocity=0.5
- joint wrist_pan_joint: limit lower=-3.14 upper=3.14 effort=0 velocity=5 -> lower=-1.57 upper=3.14 effort=0 velocity=5

Commit message: Update kinematics, joint limits, and controllers configuration

File: config/gazebo_hera.urdf (robot description, URDF)
Before this commit: robot hera, 27 links, 26 joints
Links:
- removed link base
- removed link base_scan_back
- removed link xtion_link
- removed link xtion_link_depth
- removed link xtion_link_optical
- added link base_link, mass 10.0; collision box size=0.494 0.318 0.07; visual mesh filename=package://hera_description/meshes/base/base.stl
- added link xtion, mass 0.01; collision box size=0.04 0.18 0.07; visual mesh filename=package://hera_description/meshes/sensors/asus_xtion.stl
- added link xtion_depth
- added link xtion_optical
- link backrest_link: geometry collision mesh filename=package://hera_description/meshes/manipulator/backrest.STL; visual mesh filename=package://hera_description/meshes/manipulator/backrest.STL
- link base_scan_front: geometry collision box size=0.05 0.05 0.07; visual mesh filename=package://hera_description/meshes/sensors/hokuyo_urg.dae
- link base_wheelBL: geometry collision cylinder length=0.07 radius=0.1; collision sphere radius=0.005
- link base_wheelBR: geometry collision cylinder length=0.07 radius=0.1; collision sphere radius=0.005
- link base_wheelFL: geometry collision cylinder length=0.07 radius=0.1; collision sphere radius=0.005
- link base_wheelFR: geometry collision cylinder length=0.07 radius=0.1; collision sphere radius=0.005
- link elbow_lift_link: geometry collision mesh filename=package://hera_description/meshes/manipulator/elbow_lift_co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; visual mesh filename=package://hera_description/meshes/manipulator/elbow_lift.STL
- link elbow_pan_link: geometry collision mesh filename=package://hera_description/meshes/manipulator/elbow_pan_col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; visual mesh filename=package://hera_description/meshes/manipulator/elbow_pan.STL
- link gripper_left_end_link: geometry collision mesh filename=package://hera_description/meshes/manipulator/gripper_meshe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; visual mesh filename=package://hera_description/meshes/manipulator/gripper_meshe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
- link gripper_left_link: geometry collision mesh filename=package://hera_description/meshes/manipulator/gripper_meshe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; visual mesh filename=package://hera_description/meshes/manipulator/gripper_meshe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
- link gripper_right_end_link: geometry collision mesh filename=package://hera_description/meshes/manipulator/gripper_meshe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; visual mesh filename=package://hera_description/meshes/manipulator/gripper_meshe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
- link gripper_right_link: geometry collision mesh filename=package://hera_description/meshes/manipulator/gripper_meshe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; visual mesh filename=package://hera_description/meshes/manipulator/gripper_meshe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
- link head: geometry collision box size=0.1 0.2 0.27; collision cylinder length=0.06 radius=0.065
- link manip_base_link: geometry collision mesh filename=package://hera_description/meshes/manipulator/manip_base_co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; visual mesh filename=package://hera_description/meshes/manipulator/manip_base.STL
- link manip_support_link: geometry collision mesh filename=package://hera_description/meshes/manipulator/manip_support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; visual mesh filename=package://hera_description/meshes/manipulator/manip_support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
- link shoulder_lift_link: geometry collision mesh filename=package://hera_description/meshes/manipulator/shoulder_lift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; visual mesh filename=package://hera_description/meshes/manipulator/shoulder_lift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
- link shoulder_pan_link: geometry collision mesh filename=package://hera_description/meshes/manipulator/shoulder_pan_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; visual mesh filename=package://hera_description/meshes/manipulator/shoulder_pan.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
- link torso: geometry collision box size=0.13 0.06 1.0; collision box size=0.13 0.06 1.0
- link torso_sensor_plat: geometry collision box size=0.1 0.12 0.01; visual mesh filename=package://hera_description/meshes/base/torso_sensor_plat.stl
- link wrist_lift_link: geometry collision mesh filename=package://hera_description/meshes/manipulator/wrist_lift_co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; visual mesh filename=package://hera_description/meshes/manipulator/wrist_lift.STL
- link wrist_pan_link: geometry collision mesh filename=package://hera_description/meshes/manipulator/wrist_pan_col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; visual mesh filename=package://hera_description/meshes/manipulator/wrist_pan.STL
Joints:
- removed joint base_scan_front_hokuyo_utm_joint
- removed joint joint_base_footprint_to_base
- removed joint joint_base_to_base_scan_back_hokuyo_urg
- removed joint joint_base_to_base_wheelBL
- removed joint joint_base_to_base_wheelBR
- removed joint joint_base_to_base_wheelFL
- removed joint joint_base_to_base_wheelFR
- removed joint joint_base_to_torso
- removed joint joint_torso_to_xtion_link
- removed joint joint_xtion_link_to_xtion_link_depth
- removed joint joint_xtion_link_to_xtion_link_otptical
- added joint joint_base_footprint_to_base_link: type fixed, parent base_footprint, child base_link, origin xyz=0 0 0.1
- added joint joint_base_link_to_base_scan_front_hokuyo_urg: type fixed, parent base_link, child base_scan_front, origin xyz=0.3 0 0.0 rpy=0 0 0
- added joint joint_base_link_to_base_wheelBL: type continuous, parent base_link, child base_wheelBL, origin xyz=-0.1976 0.214 0.0 rpy=0 0 0, axis 0 1 0, limit effort=30.0 velocity=0.5
- added joint joint_base_link_to_base_wheelBR: type continuous, parent base_link, child base_wheelBR, origin xyz=-0.1976 -0.214 0.0 rpy=0 0 0, axis 0 1 0, limit effort=30.0 velocity=0.5
- added joint joint_base_link_to_base_wheelFL: type continuous, parent base_link, child base_wheelFL, origin xyz=0.1976 0.214 0.0 rpy=0 0 0, axis 0 1 0, limit effort=30.0 velocity=0.5
- added joint joint_base_link_to_base_wheelFR: type continuous, parent base_link, child base_wheelFR, origin xyz=0.1976 -0.214 0.0 rpy=0 0 0, axis 0 1 0, limit effort=30.0 velocity=0.5
- added joint joint_base_link_to_torso: type fixed, parent base_link, child torso, origin xyz=0 0 0.535 rpy=0 0 0
- added joint joint_torso_sensor_plat_to_xtion: type fixed, parent torso_sensor_plat, child xtion, origin xyz=0.02 0 0.05 rpy=0 0 0
- added joint joint_xtion_to_xtion_depth: type fixed, parent xtion, child xtion_depth, origin xyz=0.0 0.049 0.016 rpy=0 0 0
- added joint joint_xtion_to_xtion_otptical: type fixed, parent xtion, child xtion_optical, origin xyz=0 0 0 rpy=-1.5707963267948966 0 -1.5707963267948966
- joint gripper_left_joint: limit lower=-1.5600 upper=0.6454 effort=0 velocity=5 -> lower=0.0 upper=0.8 effort=0 velocity=5
- joint gripper_right_joint: limit lower=-0.6454 upper=1.5600 effort=0 velocity=5 -> lower=-0.8 upper=0.0 effort=0 velocity=5
- joint joint_torso_to_torso_sensor_plat: limit lower=-1.5 upper=0.1 effort=30 velocity=0.5 -> lower=-2.0 upper=0.3 effort=30 velocity=0.5
- joint wrist_pan_joint: limit lower=-1.57 upper=3.14 effort=0 velocity=5 -> lower=-3.14 upper=3.14 effort=0 velocity=5

Commit message: Update configuration files for camera and controllers

File: config/gazebo_hera.urdf (robot description, URDF)
Before this commit: robot hera, 26 links, 25 joints
Links:
- removed link base_link
- removed link torso_sensor_plat
- removed link xtion
- removed link xtion_depth
- removed link xtion_optical
- added link base, mass 10.0; collision box size=0.494 0.318 0.07; visual mesh filename=package://hera_description/meshes/base/base.stl
- added link camera_bottom_screw_frame
- added link camera_link, mass 0.072; collision box size=0.02505 0.09 0.025; visual mesh filename=package://realsense2_description/meshes/d435.dae
- added link torso_camera_tilt, mass 0.05; visual mesh color=0.5 0.5 0.5 1 filename=package://hera_description/meshes/camera_meshes/dynamixel.s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 scale=0.001 0.001 0.001
- added link torso_connection_rod, mass 0.02; visual cylinder length=0.03 radius=0.005
- added link torso_pan_mechanism_link, mass 0.1; visual box size=0.02 0.02 0.02
- added link torso_sensor_platform, mass 0.01; collision box size=0.1 0.12 0.01; visual mesh color=0.5 0.5 0.5 1 filename=package://hera_description/meshes/camera_meshes/dynamixel.s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 scale=0.001 0.001 0.001
- link torso: geometry collision box size=0.13 0.06 1.0; collision box size=0.13 0.06 1.0
Joints:
- removed joint joint_base_footprint_to_base_link
- removed joint joint_base_link_to_base_scan_front_hokuyo_urg
- removed joint joint_base_link_to_base_wheelBL
- removed joint joint_base_link_to_base_wheelBR
- removed joint joint_base_link_to_base_wheelFL
- removed joint joint_base_link_to_base_wheelFR
- removed joint joint_base_link_to_torso
- removed joint joint_torso_sensor_plat_to_xtion
- removed joint joint_torso_to_torso_sensor_plat
- removed joint joint_xtion_to_xtion_depth
- removed joint joint_xtion_to_xtion_otptical
- added joint camera_joint: type fixed, parent torso_pan_mechanism_link, child camera_bottom_screw_frame, origin xyz=0 0 0 rpy=0 0 0
- added joint camera_link_joint: type fixed, parent camera_bottom_screw_frame, child camera_link, origin xyz=0.010600000000000002 0.0175 0.0125 rpy=0 0 0
- added joint joint_base_footprint_to_base: type fixed, parent base_footprint, child base, origin xyz=0 0 0.1
- added joint joint_base_to_base_scan_front_hokuyo_urg: type fixed, parent base, child base_scan_front, origin xyz=0.3 0 0.0 rpy=0 0 0
- added joint joint_base_to_base_wheelBL: type fixed, parent base, child base_wheelBL, origin xyz=-0.1976 0.214 0.0 rpy=0 0 0, axis 0 1 0, limit effort=30.0 velocity=0.5
- added joint joint_base_to_base_wheelBR: type fixed, parent base, child base_wheelBR, origin xyz=-0.1976 -0.214 0.0 rpy=0 0 0, axis 0 1 0, limit effort=30.0 velocity=0.5
- added joint joint_base_to_base_wheelFL: type fixed, parent base, child base_wheelFL, origin xyz=0.1976 0.214 0.0 rpy=0 0 0, axis 0 1 0, limit effort=30.0 velocity=0.5
- added joint joint_base_to_base_wheelFR: type fixed, parent base, child base_wheelFR, origin xyz=0.1976 -0.214 0.0 rpy=0 0 0, axis 0 1 0, limit effort=30.0 velocity=0.5
- added joint joint_base_to_torso: type fixed, parent base, child torso, origin xyz=0 0 0.535 rpy=0 0 0
- added joint joint_camera_pan: type revolute, parent torso_camera_tilt, child torso_pan_mechanism_link, origin xyz=0 0 0.015 rpy=0 0 0, axis 0 0 1, limit lower=-3.14 upper=3.14 effort=30 velocity=0.5
- added joint joint_camera_tilt: type revolute, parent torso_sensor_platform, child torso_connection_rod, origin xyz=0 -0.003 0.0 rpy=0 0 0, axis 0 -1 0, limit lower=-2.0 upper=0.3 effort=30 velocity=0.5
- added joint joint_torso_connection_rod_to_pan_mechanism: type fixed, parent torso_connection_rod, child torso_camera_tilt, origin xyz=0.005 0 0.05 rpy=0 0 0
- added joint joint_torso_to_sensor_platform: type fixed, parent torso, child torso_sensor_platform, origin xyz=0.085 0 0.42 rpy=0 0 0, axis 0 -1 0, limit lower=-2.0 upper=0.3 effort=30 velocity=0.5
